Commit message: Update urdf

File: assets/MOS9/MOS9_walk.urdf (robot description, URDF)
Before this commit: robot MOS91_openhand_0516, 21 links, 20 joints
Links:
- removed link body
- added link base_link, mass 5.71912; collision cylinder length=0.2 radius=0.10; visual mesh filename=meshes/body.STL
- link Lankle: mass 0.099798 -> 0.21292; geometry visual mesh filename=meshes/Lankle.STL
- link Larm: mass 0.72685 -> 0.8121; geometry collision cylinder length=0.15 radius=0.03; visual mesh filename=meshes/Larm.STL
- link Lfoot: mass 0.64424103204 -> 0.67876; geometry collision cylinder length=0.13 radius=0.03; collision cylinder length=0.16 radius=0.022
- link Lhand: mass 0.2819 -> 0.28342; geometry collision cylinder length=0.15 radius=0.02; collision sphere radius=0.024
- link Lhip: mass 0.68953 -> 0.74781; geometry visual mesh filename=meshes/Lhip.STL
- link Llap: mass 0.12125 -> 0.19423; geometry visual mesh filename=meshes/Llap.STL
- link Lleg1: mass 1.39974210238 -> 1.54675; geometry collision cylinder length=0.130 radius=0.030; visual mesh filename=meshes/Lleg1.STL
- link Lleg2: mass 0.66458 -> 0.92397; geometry collision cylinder length=0.15 radius=0.028; visual mesh filename=meshes/Lleg2.STL
- link Lshoulder: mass 0.46181 -> 0.49509; geometry visual mesh filename=meshes/Lshoulder.STL
- link Rankle: mass 0.099798 -> 0.21292; geometry visual mesh filename=meshes/Rankle.STL
- link Rarm: mass 0.72685 -> 0.8121; geometry collision cylinder length=0.15 radius=0.03; visual mesh filename=meshes/Rarm.STL
- link Rfoot: mass 0.64424103204 -> 0.67876; geometry collision cylinder length=0.13 radius=0.03; collision cylinder length=0.16 radius=0.022
- link Rhand: mass 0.28189 -> 0.28342; geometry collision cylinder length=0.15 radius=0.02; collision sphere radius=0.024
- link Rhip: mass 0.68971 -> 0.74781; geometry visual mesh filename=meshes/Rhip.STL
- link Rlap: mass 0.12125 -> 0.19423; geometry visual mesh filename=meshes/Rlap.STL
- link Rleg1: mass 1.39974202104 -> 1.54675; geometry collision cylinder length=0.130 radius=0.030; visual mesh filename=meshes/Rleg1.STL
- link Rleg2: mass 0.66458 -> 0.92397; geometry collision cylinder length=0.15 radius=0.028; visual mesh filename=meshes/Rleg2.STL
- link Rshoulder: mass 0.46181 -> 0.49509; geometry visual mesh filename=meshes/Rshoulder.STL
- link head: mass 0.31267418781 -> 0.39244; geometry collision cylinder length=0.2 radius=0.04; visual mesh filename=meshes/head.STL
- link neck: mass 0.22536239155 -> 0.49351; geometry visual mesh filename=meshes/neck.STL
Joints:
- removed joint La_Lf
- removed joint La_Lh
- removed joint Lh_Ll
- removed joint Ll1_Ll2
- removed joint Ll2_La
- removed joint Ll_Ll1
- removed joint Ls_La
- removed joint Ra_Rf
- removed joint Ra_Rh
- removed joint Rh_Rl
- removed joint Rl1_Rl2
- removed joint Rl2_Ra
- removed joint Rl_Rl1
- removed joint Rs_Ra
- removed joint b_Lh
- removed joint b_Ls
- removed joint b_Rh
- removed joint b_Rs
- removed joint b_n
- removed joint n_h
- added joint left_ankle_pitch: type revolute, parent Lleg2, child Lankle, origin xyz=0 -0.2 0.0177999999999994 rpy=0 0 0, axis 0 0 -1, limit lower=-2.1 upper=0.9
- added joint left_ankle_roll: type revolute, parent Lankle, child Lfoot, origin xyz=-0.068999999995933 0.00155678563569939 -0.0281533249166232 rpy=0 1.5707963267949 0, axis 0 0 -1, limit lower=-0.7 upper=0.7
- added joint left_elbow: type revolute, parent Larm, child Lhand, origin xyz=0.16 0.0286500000000008 -0.0299999999999989 rpy=-1.5707963267949 0 3.14159265358979, axis 0 0 -1, limit lower=-2.5 upper=2.5
- added joint left_hip_pitch: type revolute, parent base_link, child Lhip, origin xyz=-0.0150000000000001 0.0645 -0.0466 rpy=1.5707963267949 0 3.14159265358979, axis 0 0 -1, limit lower=-1.8 upper=1.8
- added joint left_hip_roll: type revolute, parent Lhip, child Llap, origin xyz=-0.027499999999988 9.99999999794776E-05 0.0609999999999988 rpy=0 1.5707963267949 0, axis 0 0 -1, limit lower=-0.25 upper=1.5707963267949
- added joint left_hip_yaw: type revolute, parent Llap, child Lleg1, origin xyz=0 -0.0629999999999796 0.0279999999999841 rpy=1.5707963267949 0 3.14159265358979, axis 0 0 -1, limit lower=-1.5707963267949 upper=1.5707963267949
- added joint left_knee: type revolute, parent Lleg1, child Lleg2, origin xyz=0.00900000000000006 0 -0.146 rpy=1.5707963267949 0 1.5707963267949, axis 0 0 -1, limit lower=-2.3 upper=1.0
- added joint left_shoulder_pitch: type revolute, parent base_link, child Lshoulder, origin xyz=-0.00999998124092416 0.105000001016346 0.192100005298829 rpy=1.5707963267949 0 0, axis 0 0 -1, limit lower=-2.0 upper=2.0
- added joint left_shoulder_roll: type revolute, parent Lshoulder, child Larm, origin xyz=0.0249999812409242 0 -0.0489999989836545 rpy=0 1.5707963267949 0, axis 0 0 -1, limit lower=-1.5707963267949 upper=1.45
- added joint neck_pitch: type fixed, parent neck, child head, origin xyz=0 -0.033 0.0475 rpy=1.5707963267949 0 0, axis 0 0 -1
- added joint neck_yaw: type fixed, parent base_link, child neck, origin xyz=-0.005 0 0.2441 rpy=0 0 0, axis 0 0 -1
- added joint right_ankle_pitch: type revolute, parent Rleg2, child Rankle, origin xyz=0 -0.2 0.0177999999999997 rpy=0 0 0, axis 0 0 -1, limit lower=-0.9 upper=2.1
- added joint right_ankle_roll: type revolute, parent Rankle, child Rfoot, origin xyz=0.0689999999999583 0 -0.0259999999999973 rpy=0 1.5707963267949 0, axis 0 0 1, limit lower=-0.7 upper=0.7
- added joint right_elbow: type revolute, parent Rarm, child Rhand, origin xyz=0.16 0.0286499999999997 0.0299999999999999 rpy=1.5707963267949 0 0, axis 0 0 -1, limit lower=-2.5 upper=2.5
- added joint right_hip_pitch: type revolute, parent base_link, child Rhip, origin xyz=-0.0150000000000001 -0.0645 -0.0466 rpy=1.5707963267949 0 3.14159265358979, axis 0 0 1, limit lower=-1.8 upper=1.8
- added joint right_hip_roll: type revolute, parent Rhip, child Rlap, origin xyz=-0.0275 0 -0.061 rpy=0 1.5707963267949 0, axis 0 0 -1, limit lower=-1.5707963267949 upper=0.25
- added joint right_hip_yaw: type revolute, parent Rlap, child Rleg1, origin xyz=0 -0.063 0.0280000000000001 rpy=1.5707963267949 0 3.14159265358979, axis 0 0 -1, limit lower=-1.5707963267949 upper=1.5707963267949
- added joint right_knee: type revolute, parent Rleg1, child Rleg2, origin xyz=-0.00900000000000004 0 -0.146 rpy=1.5707963267949 0 -1.5707963267949, axis 0 0 -1, limit lower=-1.0 upper=2.3
- added joint right_shoulder_pitch: type revolute, parent base_link, child Rshoulder, origin xyz=-0.0100000000000138 -0.105000000000124 0.192100000000112 rpy=1.5707963267949 0 -3.14159265358979, axis 0 0 -1, limit lower=-2.0 upper=2.0
- added joint right_shoulder_roll: type revolute, parent Rshoulder, child Rarm, origin xyz=-0.0250000000000136 0 -0.0489999999998756 rpy=0 1.5707963267949 0, axis 0 0 1, limit lower=-1.45 upper=1.5707963267949
