Commit message: feat: add kick sim2sim teacher actor

File: assets/PI/pi_plus.urdf (robot description, URDF)
Before this commit: robot pi_plus_24dof_250826, 25 links, 24 joints
Joints:
- joint head_pitch_joint: type fixed -> revolute
- joint head_yaw_joint: type fixed -> revolute

Commit message: Use URSoccerLab PI Plus collision primitives

File: assets/PI/pi_plus.urdf (robot description, URDF)
Before this commit: robot pi_plus_24dof_250826, 25 links, 24 joints
Links:
- link base_link: geometry collision box size=0.035 0.035 0.044; collision box size=0.045 0.075 0.045
- link head_pitch_link: geometry collision box size=0.1341606 0.1613276 0.0901892; visual mesh filename=meshes/head_pitch_link.STL
- link head_yaw_link: geometry visual mesh filename=meshes/head_yaw_link.STL
- link l_ankle_pitch_link: geometry visual mesh filename=meshes/l_ankle_pitch_link.STL
- link l_ankle_roll_link: geometry collision box size=0.1719574 0.0720036 0.082413; visual mesh filename=meshes/l_ankle_roll_link.STL
- link l_calf_link: geometry collision box size=0.0299 0.0275 0.061941; visual mesh filename=meshes/l_calf_link.STL
- link l_elbow_link: geometry collision box size=0.0235 0.0219 0.05415; visual mesh filename=meshes/l_elbow_link.STL
- link l_hip_pitch_link: geometry visual mesh filename=meshes/l_hip_pitch_link.STL
- link l_hip_roll_link: geometry collision box size=0.053 0.06 0.1176774; visual mesh filename=meshes/l_hip_roll_link.STL
- link l_shoulder_pitch_link: geometry visual mesh filename=meshes/l_shoulder_pitch_link.STL
- link l_shoulder_roll_link: geometry collision box size=0.0319 0.0235 0.10415; visual mesh filename=meshes/l_shoulder_roll_link.STL
- link l_thigh_link: geometry visual mesh filename=meshes/l_thigh_link.STL
- link l_upper_arm_link: geometry visual mesh filename=meshes/l_upper_arm_link.STL
- link l_wrist_link: geometry collision cylinder length=0.075982 radius=0.017505; collision sphere radius=0.017505
- link r_ankle_pitch_link: geometry visual mesh filename=meshes/r_ankle_pitch_link.STL
- link r_ankle_roll_link: geometry collision box size=0.1719574 0.0720036 0.082413; visual mesh filename=meshes/r_ankle_roll_link.STL
- link r_calf_link: geometry collision box size=0.0299 0.0275 0.061941; visual mesh filename=meshes/r_calf_link.STL
- link r_elbow_link: geometry collision box size=0.0235 0.0219 0.05415; visual mesh filename=meshes/r_elbow_link.STL
- link r_hip_pitch_link: geometry visual mesh filename=meshes/r_hip_pitch_link.STL
- link r_hip_roll_link: geometry collision box size=0.053 0.06 0.1176774; visual mesh filename=meshes/r_hip_roll_link.STL
- link r_shoulder_pitch_link: geometry visual mesh filename=meshes/r_shoulder_pitch_link.STL
- link r_shoulder_roll_link: geometry collision box size=0.0319 0.0235 0.10415; visual mesh filename=meshes/r_shoulder_roll_link.STL
- link r_thigh_link: geometry visual mesh filename=meshes/r_thigh_link.STL
- link r_upper_arm_link: geometry visual mesh filename=meshes/r_upper_arm_link.STL
- link r_wrist_link: geometry collision cylinder length=0.075982 radius=0.017505; collision sphere radius=0.017505
